File: Millable Version/Millable_TitanX1_GPS_Breakout.sch (EAGLE design)
At the start: 21 parts, among them U1 TITAN_X1_GPS, U2 6.8MM_COIN_CELL

Commit message: Adding example firmware, docs, and Qwiic board.
Parts:
- J1, J4: value (none) -> SMD
- J8: value (none) -> PTH
